File: ergogen/output/pcbs/knuckles_wireless.kicad_pcb (KiCad board)
At the start: 2 copper layers, 130.3 x 107.9 mm, 120 parts

Commit message: chore: more renaming
Other:
- board text added: "knuckles v1.0"
- board text removed: "Zeph v1.0"
Changed lines of the file:
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@@
   (paper "A3")
   (title_block
-    (title "zeph_wireless")
+    (title "knuckles_wireless")
     (date "2025-03-17")
     (rev "0.2")
@@
   (segment (start 215.90430500000002 86.635) (end 215.303695 86.635) (width 0.25) (layer "B.Cu"))
   (segment (start 215.303695 86.635) (end 214.798695 87.14) (width 0.25) (layer "B.Cu"))
-  (gr_text "Zeph v1.0"
+  (gr_text "knuckles v1.0"
     (at 137 107.4 0)
     (layer "F.SilkS" )
@@
     )
   )
-  (gr_text "Zeph v1.0"
+  (gr_text "knuckles v1.0"
     (at 137 107.4 0)
     (layer "B.SilkS" )
