File: ergogen/output/pcbs/knuckles_wireless.kicad_pcb (KiCad board)
At the start: 2 copper layers, 130.3 x 107.9 mm, 120 parts

Commit message: feat: default to compact 18.5 mm layout and refresh generated boards
Parts:
- removed DISP1: , ceoloide:display_nice_view
- added ART1: , knuckles_artwork_badge, F.Cu at (211.3, 105.8)
- added ART2: , knuckles_artwork_wordmark, F.Cu at (138.0, 105.4)
Routing:
- net SDA: track 3.50 -> 0.00 mm
- net SCL: track 3.50 -> 0.00 mm
- net GND: track 3.50 -> 0.00 mm
- net CS: track 3.50 -> 0.00 mm
Other:
- board text added: "v1.0"
- board text removed: "knuckles v1.0"
