File: hardware/integrated-controller/output/core.kicad_sch (KiCad schematic)
At the start: 17 parts, among them J1 TYPE-C-31-M-12, J3 SM04B-SRSS-TB(LF)(SN), J4 Matrix bring-up header, J5 SWD pogo interface, SW2 SKRPANE010, U1 MDBT50Q-1MV2, U4 USBLC6-2SC6

Commit message: Integrate controller layouts and validate power and firmware design
Parts:
- added C13: 100nF, Knuckles:C_0603_1608Metric, symbol Knuckles:C13
- added R18: 27R, Knuckles:R_0603_1608Metric, symbol Knuckles:R18
- added R19: 27R, Knuckles:R_0603_1608Metric, symbol Knuckles:R19
- C2: value 1uF -> 22uF; footprint Knuckles:C_0603_1608Metric -> Knuckles:C_0805_2012Metric; LCSC C15849 -> C45783
- C3: value 100nF -> 4.7uF; LCSC C14663 -> C19666
- J5: footprint Knuckles:Tag-Connect_TC2030-IDC-NL_2x03_P1.27mm_Vertical -> Knuckles:SWD_2x3_P1.27_NoHoles
Connections:
- net GND: now also C13.2 (C2)
- net USB_DN: now also R19.1 (R1); no longer U1.34 (D-)
- net USB_DP: now also R18.1 (R1); no longer U1.35 (D+)
- net VBUS: now also C13.1 (C1)
- net PMIC_SCL: now reaches U1.16 (P0.27)
- net PMIC_SDA: now reaches U1.19 (P0.26)
- net CHG_ALLOW: now reaches U1.24 (P0.08)
- net CHG_STAT1 renamed CHG_INT_N
- net CHG_STAT2 renamed CHG_PG_N
- new net USB_MCU_DN: R19.2 (R2), U1.34 (D-)
- new net USB_MCU_DP: R18.2 (R2), U1.35 (D+)
- no-connect marks 33 -> 30
