File: hardware/integrated-controller/output/knuckles_controller.kicad_sch (KiCad schematic)
At the start: 0 parts

Commit message: Integrate controller layouts and validate power and firmware design
Other:
- note added: "1S 4.2V LiPo • 110–500mAh with matching firmware battery profile"
- note added: "BQ25186: programmable current / 12-hour timer / USB suspend"
- note added: "CHARGING DISABLED: R12 interlock + firmware control; verify cell/NTC"
- note added: "Prototype circuitry; not a fabrication release"
- note removed: "1S 4.2V LiPo • 110mAh baseline; larger capacities supported"
- note removed: "CHARGING DISABLED: fit charge-enable R12 only after cell/NTC checks"
- note removed: "Default charge target 20mA; 100mA input limit"
- note removed: "Prototype circuitry; not a fabrication release or a complete keyboard layout"
