File: hardware/integrated-controller/output/knuckles_controller.kicad_pcb (KiCad board)
At the start: 2 copper layers, 45 x 55 mm, 44 parts, among them J1 TYPE-C-31-M-12, J2 S2B-PH-SM4-TB(LF)(SN), J3 SM04B-SRSS-TB(LF)(SN), J4 Matrix bring-up header, J5 SWD pogo interface, J6 External 10k NTC pads, Q1 AO3401A, Q2 2N7002, SW1 MSK12C02, SW2 SKRPANE010, U1 MDBT50Q-1MV2, U2 BQ25185DLHR, U3 TPS63031DSKR, U4 USBLC6-2SC6

Commit message: Integrate controller layouts and validate power and firmware design
Parts:
- removed C7: 47pF, Knuckles:C_0603_1608Metric
- added C13: 100nF, Knuckles:C_0603_1608Metric, F.Cu at (26.0, 43.5)
- added Q3: 2N7002, Knuckles:SOT-23, F.Cu at (25.0, 39.0)
- added R18: 27R, Knuckles:R_0603_1608Metric, F.Cu at (26.0, 18.5)
- added R19: 27R, Knuckles:R_0603_1608Metric, F.Cu at (29.0, 18.5)
- C10, C11, C6, C8: value 10uF -> 22uF; footprint Knuckles:C_0603_1608Metric -> Knuckles:C_0805_2012Metric
- C2: value 1uF -> 22uF; footprint Knuckles:C_0603_1608Metric -> Knuckles:C_0805_2012Metric
- C3: value 100nF -> 4.7uF
- C4, C5: value 1uF -> 2.2uF
- J5: footprint Knuckles:Tag-Connect_TC2030-IDC-NL_2x03_P1.27mm_Vertical -> Knuckles:SWD_2x3_P1.27_NoHoles
- R10: value 12k -> 100k
- R15, R16: value 1M -> 10k
- R8: value 15k -> 10k
- R9: value 12k -> 10k
- SW1: value MSK12C02 -> SSSS811101; footprint Knuckles:MSK12C02 -> Knuckles:SSSS811101
- U2: value BQ25185DLHR -> BQ25186DLHR
- moved J6 26.0 mm to (38.0, 53.0)
- moved C3 25.1 mm to (31.5, 16.5)
- moved R2 16.8 mm to (15.0, 51.0)
- moved R1 13.0 mm to (15.0, 47.0)
- moved C5 3.61 mm to (32.0, 39.0)
- moved R10 2.24 mm to (32.0, 44.0)
- moved J1 2.00 mm to (22.5, 52.0), turned to 0 degrees
- moved R13 2.00 mm to (27.0, 27.0)
- moved U4 1.50 mm to (22.5, 43.5)
- moved R11 1.30 mm to (26.3, 34.0)
Connections:
- net CHG_STAT1 renamed CHG_INT_N
- net CHG_STAT2 renamed CHG_PG_N
- R10 pad 1: VSET_MID -> CHG_ALLOW
- R12 pad 2: GND -> CHG_DRAIN
- R8 pad 1: CHG_ISET -> +3V3
- R8 pad 2: GND -> PMIC_SDA
- R9 pad 1: CHG_VSET -> +3V3
- R9 pad 2: VSET_MID -> PMIC_SCL
- U1 pad 16: (no net) -> PMIC_SCL
- U1 pad 19: (no net) -> PMIC_SDA
- U1 pad 24: (no net) -> CHG_ALLOW
- U1 pad 34: USB_DN -> USB_MCU_DN
- U1 pad 35: USB_DP -> USB_MCU_DP
- U2 pad 7: CHG_VSET -> PMIC_SDA
- U2 pad 8: CHG_ISET -> PMIC_SCL
Other:
- board text added: "KNUCKLES CTRL 0.2"
- board text removed: "KNUCKLES CTRL 0.1"

Commit message: Route and validate integrated keyboard variants
Parts:
- L1: value 1.5uH SWPA3015S1R5MT -> 1.5uH SWPA3015S1R5NT
