File: hardware/integrated-controller/output/power.kicad_sch (KiCad schematic)
At the start: 27 parts, among them J2 S2B-PH-SM4-TB(LF)(SN), J6 External 10k NTC pads, Q1 AO3401A, Q2 2N7002, SW1 MSK12C02, U2 BQ25185DLHR, U3 TPS63031DSKR

Commit message: Integrate controller layouts and validate power and firmware design
Parts:
- removed C7: 47pF, Knuckles:C_0603_1608Metric, symbol Knuckles:C7
- added Q3: 2N7002, Knuckles:SOT-23, symbol Knuckles:Q3
- C10, C11, C6, C8: value 10uF -> 22uF; footprint Knuckles:C_0603_1608Metric -> Knuckles:C_0805_2012Metric; LCSC C19702 -> C45783
- C4, C5: value 1uF -> 2.2uF; LCSC C15849 -> C23630
- R10: value 12k -> 100k; LCSC C22790 -> C25803
- R15, R16: value 1M -> 10k; LCSC C22935 -> C25804
- R8: value 15k -> 10k; LCSC C22809 -> C25804
- R9: value 12k -> 10k; LCSC C22790 -> C25804
- SW1: value MSK12C02 -> SSSS811101; footprint Knuckles:MSK12C02 -> Knuckles:SSSS811101; LCSC C431540 -> C109335
- U2: value BQ25185DLHR -> BQ25186DLHR; LCSC C19725033 -> C44639442
Connections:
- net +3V3: now also R8.1 (R1), R9.1 (R1)
- net GND: now also Q3.2 (S); no longer R12.2 (R2), R8.2 (R2)
- net CHG_ISET renamed PMIC_SCL
- net PMIC_SCL: now also R9.2 (R2); no longer R8.1 (R1)
- net CHG_STAT1 renamed CHG_INT_N
- net CHG_STAT2 renamed CHG_PG_N
- net CHG_VSET renamed PMIC_SDA
- net PMIC_SDA: now also R8.2 (R2); no longer R9.1 (R1)
- net VSET_MID renamed CHG_ALLOW
- net CHG_ALLOW: now also Q3.1 (G); no longer R9.2 (R2)
- new net CHG_DRAIN: Q3.3 (D), R12.2 (R2)

Commit message: Route and validate integrated keyboard variants
Parts:
- L1: value 1.5uH SWPA3015S1R5MT -> 1.5uH SWPA3015S1R5NT; LCSC C83434 -> C56594
