File: hardware/integrated-controller/output/integrated/18.5/knuckles_integrated_left.kicad_pcb (KiCad board)
At the start: 4 copper layers, 130.3 x 107.9 mm, 103 parts, among them J1 TYPE-C-31-M-12, J2 S2B-PH-SM4-TB(LF)(SN), J5 SWD pogo interface, J6 External 10k NTC pads, Q1 AO3401A, Q2 2N7002, Q3 2N7002, SW1 SSSS811101, SW2 SKRPANE010, U1 MDBT50Q-1MV2, U2 BQ25186DLHR, U3 TPS63031DSKR, U4 USBLC6-2SC6

Commit message: Route and validate integrated keyboard variants
Parts:
- L1: value 1.5uH SWPA3015S1R5MT -> 1.5uH SWPA3015S1R5NT
- R13, R7, R8, R9: moved to B.Cu
- moved R6 18.1 mm to (219.6, 78.0)
- moved R7 13.0 mm to (206.0, 88.0), turned to 180 degrees
- moved SW2 10.7 mm to (217.6, 65.4)
- moved R9 9.00 mm to (212.0, 84.0), turned to 180 degrees
- moved J5 7.50 mm to (212.0, 57.5)
- moved C11 7.42 mm to (210.9, 86.6), turned to 90 degrees
- moved C10 6.34 mm to (206.9, 86.6)
- moved R19 6.21 mm to (206.8, 108.4)
- moved C9 5.27 mm to (211.4, 90.0)
- moved L1 4.84 mm to (204.2, 90.0), turned to 90 degrees
- moved C8 2.60 mm to (205.2, 93.5), turned to -90 degrees
- moved C3 2.00 mm to (204.0, 107.0)
- moved R18 1.55 mm to (208.5, 108.4)
- moved R13 1.50 mm to (206.0, 93.9)
- moved R8 1.00 mm to (208.0, 76.0), turned to 180 degrees
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Routing:
- net USB_DN: track 0.00 -> 80.1 mm, vias 0 -> 4
- net USB_DP: track 0.00 -> 75.2 mm, vias 0 -> 4
- net SYS: track 0.00 -> 49.0 mm, vias 0 -> 4
- net GND: track 0.00 -> 46.2 mm, vias 0 -> 22
- net VBAT: track 0.00 -> 33.2 mm, vias 0 -> 2
- net VBUS: track 0.00 -> 21.0 mm, vias 0 -> 3
- net CHG_INT_N: track 0.00 -> 18.0 mm, vias 0 -> 1
- net C1: track 0.00 -> 17.9 mm, vias 0 -> 2
- net REG_EN: track 0.00 -> 13.1 mm, vias 0 -> 1
- net USB_CC2: track 0.00 -> 9.29 mm, vias 0 -> 1
- net +3V3: track 0.00 -> 8.06 mm, vias 0 -> 1
- net SW_L2: track 0.00 -> 2.86 mm
- net SW_L1: track 0.00 -> 2.86 mm
- net USB_MCU_DP: track 0.00 -> 2.38 mm, vias 0 -> 1
- net CHG_EN_N: track 0.00 -> 2.31 mm, vias 0 -> 1
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- added copper zone on In1.Cu, net GND
- added copper zone on In2.Cu, net GND
