File: hardware/integrated-controller/output/integrated/18.5/knuckles_integrated_right-power.kicad_sch (KiCad schematic)
At the start: 27 parts, among them J2 S2B-PH-SM4-TB(LF)(SN), J6 External 10k NTC pads, Q1 AO3401A, Q2 2N7002, Q3 2N7002, SW1 SSSS811101, U2 BQ25186DLHR, U3 TPS63031DSKR

Commit message: Route and validate integrated keyboard variants
Parts:
- L1: value 1.5uH SWPA3015S1R5MT -> 1.5uH SWPA3015S1R5NT; LCSC C83434 -> C56594
