File: hardware/integrated-controller/output/integrated/19.5/knuckles_integrated_left.kicad_pcb (KiCad board)
At the start: 4 copper layers, 137.3 x 113.5 mm, 103 parts, among them J1 TYPE-C-31-M-12, J2 S2B-PH-SM4-TB(LF)(SN), J5 SWD pogo interface, J6 External 10k NTC pads, Q1 AO3401A, Q2 2N7002, Q3 2N7002, SW1 SSSS811101, SW2 SKRPANE010, U1 MDBT50Q-1MV2, U2 BQ25186DLHR, U3 TPS63031DSKR, U4 USBLC6-2SC6

Commit message: Route and validate integrated keyboard variants
Parts:
- L1: value 1.5uH SWPA3015S1R5MT -> 1.5uH SWPA3015S1R5NT
- R13, R7, R8, R9: moved to B.Cu
- moved R6 18.1 mm to (225.2, 75.5)
- moved R7 13.0 mm to (211.5, 85.5), turned to 180 degrees
- moved SW2 10.7 mm to (223.2, 62.9)
- moved R9 9.00 mm to (217.5, 81.5), turned to 180 degrees
- moved J5 7.50 mm to (217.5, 55.0)
- moved C11 7.42 mm to (216.5, 84.1), turned to 90 degrees
- moved C10 6.34 mm to (212.5, 84.1)
- moved R19 6.21 mm to (212.3, 105.9)
- moved C9 5.27 mm to (217.0, 87.5)
- moved L1 4.84 mm to (209.7, 87.5), turned to 90 degrees
- moved C8 2.60 mm to (210.8, 91.0), turned to -90 degrees
- moved C3 2.00 mm to (209.5, 104.5)
- moved R18 1.55 mm to (214.0, 105.9)
- moved R13 1.50 mm to (211.5, 91.4)
- moved R8 1.00 mm to (213.5, 73.5), turned to 180 degrees
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Routing:
- net USB_DN: track 0.00 -> 80.1 mm, vias 0 -> 4
- net USB_DP: track 0.00 -> 75.2 mm, vias 0 -> 4
- net SYS: track 0.00 -> 49.0 mm, vias 0 -> 4
- net GND: track 0.00 -> 46.2 mm, vias 0 -> 22
- net VBAT: track 0.00 -> 33.2 mm, vias 0 -> 2
- net CHG_INT_N: track 0.00 -> 18.0 mm, vias 0 -> 1
- net REG_EN: track 0.00 -> 13.1 mm, vias 0 -> 1
- net VBUS: track 0.00 -> 12.4 mm, vias 0 -> 3
- net +3V3: track 0.00 -> 8.06 mm, vias 0 -> 1
- net SW_L2: track 0.00 -> 2.86 mm
- net SW_L1: track 0.00 -> 2.86 mm
- net USB_MCU_DP: track 0.00 -> 2.38 mm, vias 0 -> 1
- net CHG_EN_N: track 0.00 -> 2.31 mm, vias 0 -> 1
- net USB_MCU_DN: track 0.00 -> 1.95 mm, vias 0 -> 1
- net PMIC_SDA: track 0.00 -> 1.81 mm, vias 0 -> 1
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- added copper zone on In1.Cu, net GND
- added copper zone on In2.Cu, net GND
