File: hardware/integrated-controller/output/integrated/19.5/knuckles_integrated_right.kicad_pcb (KiCad board)
At the start: 4 copper layers, 137.3 x 113.5 mm, 106 parts, among them J1 TYPE-C-31-M-12, J2 S2B-PH-SM4-TB(LF)(SN), J3 SM04B-SRSS-TB(LF)(SN), J5 SWD pogo interface, J6 External 10k NTC pads, Q1 AO3401A, Q2 2N7002, Q3 2N7002, SW1 SSSS811101, SW2 SKRPANE010, U1 MDBT50Q-1MV2, U2 BQ25186DLHR, U3 TPS63031DSKR, U4 USBLC6-2SC6

Commit message: Route and validate integrated keyboard variants
Parts:
- L1: value 1.5uH SWPA3015S1R5MT -> 1.5uH SWPA3015S1R5NT
- R13, R7, R8, R9: moved to B.Cu
- R18, R19: moved to F.Cu
- moved R19 15.8 mm to (116.0, 91.1)
- moved R7 15.0 mm to (110.0, 85.5), turned to 180 degrees
- moved R18 14.5 mm to (114.1, 91.1)
- moved R6 10.0 mm to (118.2, 75.5)
- moved C11 9.80 mm to (117.5, 84.1), turned to 90 degrees
- moved R9 9.00 mm to (110.6, 81.5), turned to 180 degrees
- moved J5 7.50 mm to (110.6, 55.0)
- moved C4 7.00 mm to (118.1, 69.5)
- moved C5 7.00 mm to (111.1, 69.5)
- moved C8 6.75 mm to (111.8, 91.0)
- moved C9 5.27 mm to (118.0, 87.5)
- moved C10 5.03 mm to (113.5, 84.1), turned to 90 degrees
- moved L1 4.84 mm to (110.8, 87.5), turned to 90 degrees
- moved SW2 1.10 mm to (116.2, 62.9)
- moved R8 1.00 mm to (114.6, 73.5), turned to 180 degrees
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Routing:
- net USB_DP: track 0.00 -> 49.8 mm, vias 0 -> 5
- net SYS: track 0.00 -> 49.0 mm, vias 0 -> 4
- net USB_DN: track 0.00 -> 48.2 mm, vias 0 -> 5
- net GND: track 0.00 -> 43.4 mm, vias 0 -> 22
- net VBAT: track 0.00 -> 26.6 mm, vias 0 -> 2
- net VBUS: track 0.00 -> 18.2 mm, vias 0 -> 3
- net CHG_INT_N: track 0.00 -> 11.6 mm, vias 0 -> 1
- net +3V3: track 0.00 -> 8.06 mm, vias 0 -> 1
- net REG_EN: track 0.00 -> 4.23 mm, vias 0 -> 1
- net SW_L2: track 0.00 -> 2.86 mm
- net SW_L1: track 0.00 -> 2.86 mm
- net CHG_EN_N: track 0.00 -> 2.31 mm, vias 0 -> 1
- net USB_MCU_DP: track 0.00 -> 2.26 mm
- net USB_MCU_DN: track 0.00 -> 2.04 mm
- net TPS_SCL: track 0.00 -> 1.68 mm, vias 0 -> 1
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- added copper zone on In1.Cu, net GND
- added copper zone on In2.Cu, net GND
